Commit message: with two grippers version

File: config/g1_29dof.ros2_control.xacro (robot description, xacro)
@@ -106,4 +106,18 @@
                 <state_interface name="velocity"/>
             </joint>
+            <joint name="left_gripper_pinion_joint">
+                <command_interface name="position"/>
+                <state_interface name="position">
+                  <param name="initial_value">${initial_positions['left_gripper_pinion_joint']}</param>
+                </state_interface>
+                <state_interface name="velocity"/>
+            </joint>
+            <joint name="right_gripper_pinion_joint">
+                <command_interface name="position"/>
+                <state_interface name="position">
+                  <param name="initial_value">${initial_positions['right_gripper_pinion_joint']}</param>
+                </state_interface>
+                <state_interface name="velocity"/>
+            </joint>
         </ros2_control>
     </xacro:macro>

File: config/g1_29dof.urdf.xacro (robot description, xacro)
@@ -3,5 +3,5 @@
     <xacro:arg name="initial_positions_file" default="initial_positions.yaml" />
     <!-- Import g1_29dof urdf file -->
-    <xacro:include filename="$(find g1_description)/urdf/g1_29dof.urdf" />
+    <xacro:include filename="$(find g1_description)/urdf/g1_gripper.urdf.xacro" />
     <!-- Import control_xacro -->
     <xacro:include filename="g1_29dof.ros2_control.xacro" />
